File: hardware/control_board/BORC_v2_control_board.brd (EAGLE design)
At the start: 75 x 74.8 mm, 175 parts, among them J1 USB Female Type C Connector, J2 QWIIC_RIGHT_ANGLE, J3 M20-8900405, J5 S2B-XH-A(LF)(SN), Q1 UMT3904T106, Q10 BSS138PW,115, Q11 SSM3J374R,LF, Q16 UMT3904T106, Q3 BSS138PW,115, Q4 UMT3904T106, Q5 SSM3J374R,LF, Q6 SSM3K376R,LF, Q7 SSM3J374R,LF, Q9 BSS138PW,115, SW1 SPST_TACT-KMR2, U1 ATMEGA1284P-MU, U11 INA219AIDCNR, U12 SY6982C, U2 SHT40-BD1B, U3 PCA9685, U4 MCP1703CB, U5 RPM5.0-3.0, U6 915MHz, U7 AT25F512BJEDEC_3.9MM, U8 FT231XQ-R, Y1 16 MHz

Commit message: v2.1 - bug fixes and design update
Parts:
- removed C27, C5: 0.1uF, Adafruit Feather 32u4 Bluefruit LE:MICROBUILDER__0402MP
- removed C28, C29: 47uF, SparkFun-Passives:0805
- removed C31: 470nF, Adafruit Feather 32u4 Bluefruit LE:MICROBUILDER__0402MP
- removed C32, C33: 10uF, SparkFun-Passives:0805
- removed L1: SRN5040TA-2R2M, SRN5040TA-2R2M:4.95X4.95MM
- removed R34: 330, Adafruit Feather 32u4 Bluefruit LE:MICROBUILDER__0402MP
- removed R37, R38: 10K, Adafruit Feather 32u4 Bluefruit LE:MICROBUILDER__0402MP
- removed TP27, TP36, TP37: RX, Adafruit Feather 32u4 Bluefruit LE:MICROBUILDER_TESTPOINT_ROUND_1MM
- removed U12: SY6982C, SY6982C:QFN3X3-16
- added C20, C22: 10uF, Adafruit Feather 32u4 Bluefruit LE:MICROBUILDER__0402MP
- added D4: MBR260HW, microbuilder:SOD-123
- added Q2: SSM3J374R,LF, MOSFETs:SOT23-3
- added R31, R32, R33: 10K, Adafruit Feather 32u4 Bluefruit LE:MICROBUILDER__0402MP
- added TP3, TP4: RX, Adafruit Feather 32u4 Bluefruit LE:MICROBUILDER_TESTPOINT_ROUND_1MM
- added U9: MCP73833T-AMI/MF, microbuilder:DFN10_3X3MM
- C23: value 0.1uF -> 10uF
- D1: value MBR120 -> STPS140Z
- Q1: value UMT3904T106 -> SSM3J374R,LF; device SOT65P210X100-3N:SOT65P210X100-3N -> MOSFETs:SOT23-3
- Q6: value SSM3K376R,LF -> UMT3904T106; device MOSFETs:SOT23-3 -> SOT65P210X100-3N:SOT65P210X100-3N
- R18: value 470k -> 10M
- R27: value 1.69M -> 1K
- R36: value 10K -> 1K
- U5: value RPM5.0-3.0 -> POLOLU_STEPUP_U3V40F5; device RPM5.0-3.0:CONV_RPM5.0-3.0 -> Pololu Step Up Vregs:POLOLU_STEPUP_U3V40X
- moved Q1 35.6 mm to (10.1, 50.4), turned to 0 degrees
- moved C11 18.7 mm to (35.9, 24.7), turned to 180 degrees
- moved C13 18.6 mm to (39.1, 24.7), turned to 0 degrees
- moved R27 18.0 mm to (46.4, 38.7), turned to 270 degrees
- moved TP45 17.4 mm to (33.7, 26.7)
- moved TP13 17.3 mm to (11.2, 33.5)
- moved R19 16.5 mm to (35.9, 26.3), turned to 180 degrees
- moved R20 16.4 mm to (39.1, 26.3), turned to 0 degrees
- moved Q7 15.4 mm to (62.1, 25.4), turned to 90 degrees
- moved Q5 15.2 mm to (66.0, 24.2), turned to 180 degrees
- moved TP46 15.1 mm to (40.0, 25.8)
- moved R21 14.3 mm to (35.9, 28.0), turned to 0 degrees
- moved R22 14.1 mm to (39.1, 28.0), turned to 180 degrees
- moved TP48 13.7 mm to (49.8, 34.6)
- moved Q6 13.5 mm to (48.3, 41.4)
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Connections:
- removed net ACC_POWER: R34.2, TP37.P$1, U1.24
- removed net GND0: C2.2, C9.2, Q1.3, R18.2, R5.2, TP36.P$1
- removed net LX: C23.1, L1.P$2, U12.LX
- removed net N$19: C23.2, U12.BST
- removed net N$21: Q1.1, R34.1
- removed net N$22: C30.2, U12.BD@1, U12.BD@2
- removed net N$23: LED14.-, U12.STAT
- removed net N$25: LED14.+, R35.2
- removed net N$26: C31.1, U12.TIM
- removed net N$28: R37.2, R38.1, U12.NTC
- removed net N$30: R27.2, U5.E5
- removed net VBAT-: J5.1, Q6.3, TP27.P$1
- new net DISPLAY_3V3: J2.2, Q1.3, TP40.P$1
- new net LED_5V: C20.1, C22.1, LED10.3, LED11.3, LED4.3, LED7.3, LED8.3, LED9.3, Q2.3, R45.1, R47.1
- new net LED_POWER: R27.2, TP3.P$1, U1.24
- new net N$16: LED14.-, R35.1
- new net N$18: Q2.1, Q6.3, R32.2
- new net N$20: Q6.1, R27.1, R31.1
- new net N$9: R35.2, U9.P$3
- net 5V: now also D4.C, Q2.2, R32.1, U5.P$6, U5.VOUT; no longer C33.1, LED10.3, LED11.3, LED4.3, LED7.3, LED8.3, LED9.3, R45.1, R47.1, U5.A5, U5.B5, U5.C5
- net CHANNEL_A: now also U1.12; no longer U1.11
- net CHANNEL_B: now also U1.11; no longer U1.12
- net DISPLAY_POWER: now also Q1.1, R33.2, TP4.P$1; no longer J2.2, TP40.P$1
- net GND: now also C2.2, C20.2, C22.2, C23.2, C24.2, C30.2, C9.2, D4.A, J5.1, R18.2, R31.2, R5.2, U5.GND@1, U5.GND@2, U5.P$4, U5.P$5, U9.P$5; no longer C24.1, C27.1, C28.2, C29.2, C30.1, C31.2, C32.2, C33.2, C5.2, Q1.2, R27.1, R37.1, U12.PGND, U12.SGND, U5.A3, U5.A4, U5.B1, U5.B2, U5.B3, U5.B4, U5.C2, U5.C3, U5.C4, U5.D2, U5.D3, U5.D4, U5.D5, U5.E3, U5.E4
- net N$27: now also U9.P$6; no longer U12.ICHG
- net PWR_IN: now also C23.1, C24.1, Q7.3, U5.P$2, U5.P$3, U5.VIN@1, U5.VIN@2; no longer C32.1, C5.1, Q7.2, U5.A1, U5.A2
- net VBAT: now also C30.1, U9.P$10, U9.P$9; no longer C27.2, C28.1, C29.1, Q6.1, U12.BAT
- net VBUS_FUSED: now also LED14.+, U9.P$1, U9.P$2; no longer C24.2, L1.P$1, R35.1, R38.2, U12.EN, U12.ILIM
- net VCC: now also Q1.2, R33.1
- net VIN: now also Q7.2; no longer Q7.3
Routing:
- net LED_5V: track 0.00 -> 249.5 mm, vias 0 -> 9
- net 5V: track 251.9 -> 38.2 mm, vias 8 -> 1
- net N$23: track 53.1 -> 0.00 mm, vias 2 -> 0
- net GND0: track 47.7 -> 0.00 mm, vias 2 -> 0
- net N$9: track 0.00 -> 47.4 mm, vias 0 -> 2
- net LED_POWER: track 0.00 -> 35.0 mm, vias 0 -> 2
- net N$31: track 2.65 -> 28.4 mm, vias 0 -> 2
- net PWR_IN: track 0.00 -> 24.7 mm
- net VBAT: track 39.3 -> 61.6 mm, vias 2 -> 1
- net VBUS_FUSED: track 162.1 -> 140.2 mm
- net CHANNEL_A: track 48.6 -> 27.1 mm
- net ACC_POWER: track 20.3 -> 0.00 mm, vias 2 -> 0
- net CHANNEL_B: track 48.8 -> 32.4 mm
- net VIN: track 106.5 -> 94.1 mm
- net DISPLAY_3V3: track 0.00 -> 11.7 mm, vias 0 -> 1
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- added copper zone on layer 1, net 5V
- added copper zone on layer 1, net VBUS_FUSED
Other:
- board text added: "v2.1 2024-02-04"
- board text removed: "v2.0 2023-11-10"
