File: hardware/control_board/BORC_v2_control_board.sch (EAGLE design)
At the start: 175 parts, among them J1 USB Female Type C Connector, J2 QWIIC_RIGHT_ANGLE, J3 M20-8900405, J5 S2B-XH-A(LF)(SN), Q1 UMT3904T106, Q10 BSS138PW,115, Q11 SSM3J374R,LF, Q16 UMT3904T106, Q3 BSS138PW,115, Q4 UMT3904T106, Q5 SSM3J374R,LF, Q6 SSM3K376R,LF, Q7 SSM3J374R,LF, Q9 BSS138PW,115, SW1 SPST_TACT-KMR2, U1 ATMEGA1284P-MU, U11 INA219AIDCNR, U12 SY6982C, U2 SHT40-BD1B, U3 PCA9685, U4 MCP1703CB, U5 RPM5.0-3.0, U6 915MHz, U7 AT25F512BJEDEC_3.9MM, U8 FT231XQ-R, Y1 16 MHz

Commit message: v2.1 - bug fixes and design update
Parts:
- removed C27, C5: 0.1uF, Adafruit Feather 32u4 Bluefruit LE:MICROBUILDER_CAP_CERAMIC_0402MP
- removed C28, C29: 47uF, SparkFun-Passives:CAP0805
- removed C31: 470nF, Adafruit Feather 32u4 Bluefruit LE:MICROBUILDER_CAP_CERAMIC_0402MP
- removed C32, C33: 10uF, SparkFun-Passives:CAP0805
- removed L1: SRN5040TA-2R2M, SRN5040TA-2R2M:SRN5040TA-2R2M
- removed R34: 330, Adafruit Feather 32u4 Bluefruit LE:MICROBUILDER_RESISTOR_0402MP
- removed R37, R38: 10K, Adafruit Feather 32u4 Bluefruit LE:MICROBUILDER_RESISTOR_0402MP
- removed TP27, TP36, TP37: RX, Adafruit Feather 32u4 Bluefruit LE:MICROBUILDER_TESTPOINTROUND1MM
- removed U12: SY6982C, SY6982C:SY6982C
- added C20, C22: 10uF, Adafruit Feather 32u4 Bluefruit LE:MICROBUILDER_CAP_CERAMIC_0402MP
- added D4: MBR260HW, microbuilder:DIODE-SCHOTTKYSOD-123
- added Q2: SSM3J374R,LF, MOSFETs:MOSFET-PCH-BSS84
- added R31, R32, R33: 10K, Adafruit Feather 32u4 Bluefruit LE:MICROBUILDER_RESISTOR_0402MP
- added TP3, TP4: RX, Adafruit Feather 32u4 Bluefruit LE:MICROBUILDER_TESTPOINTROUND1MM
- added U9: MCP73833T-AMI/MF, microbuilder:MCP73833DFN
- C23: value 0.1uF -> 10uF
- C24: MPN GRM155R61A106ME11D -> GRM155R71H104KE14D
- D1: value MBR120 -> STPS140Z
- Q1: value UMT3904T106 -> SSM3J374R,LF; device SOT65P210X100-3N:UMT3904T106 -> MOSFETs:MOSFET-PCH-BSS84; MPN UMT3904T106 -> SSM3J374R,LF
- Q6: value SSM3K376R,LF -> UMT3904T106; device MOSFETs:MOSFET-NCH-BSS138 -> SOT65P210X100-3N:UMT3904T106; MPN SSM3K376R,LF -> UMT3904T106
- R18: value 470k -> 10M; MPN RC0402FR-13470KL -> RC0402FR-0710ML
- R27: value 1.69M -> 1K; MPN RC0402FR-071M69L -> RC0402FR-071KL
- R36: value 10K -> 1K; MPN RC0402FR-7W10KL -> RC0402FR-071KL
- U5: value RPM5.0-3.0 -> POLOLU_STEPUP_U3V40F5; device RPM5.0-3.0:RPM5.0-3.0 -> Pololu Step Up Vregs:POLOLU_STEPUP_U3V40X; MPN RPM5.0-3.0 -> U3V40F5
Connections:
- removed net ACC_POWER: R34.2, TP37.P$1, U1.PC5_[TDI/PCINT21]
- removed net GND0: C2.2, C9.2, Q1.C, R18.2, R5.2, TP36.P$1
- removed net LX: C23.1, L1.2, U12.LX
- removed net N$19: C23.2, U12.BST
- removed net N$21: Q1.B, R34.1
- removed net N$22: C30.2, U12.BD
- removed net N$23: LED14.-, U12.STAT
- removed net N$25: LED14.+, R35.2
- removed net N$26: C31.1, U12.TIM
- removed net N$28: R37.2, R38.1, U12.NTC
- removed net N$30: R27.2, U5.TRIM
- removed net VBAT-: J5.1, Q6.D, TP27.P$1
- new net DISPLAY_3V3: J2.2, Q1.D1, TP40.P$1
- new net LED_5V: C20.1, C22.1, LED10.VDD, LED11.VDD, LED4.VDD, LED7.VDD, LED8.VDD, LED9.VDD, Q2.D1, R45.1, R47.1
- new net LED_POWER: R27.2, TP3.P$1, U1.PC5_[TDI/PCINT21]
- new net N$16: LED14.-, R35.1
- new net N$18: Q2.G1, Q6.C, R32.2
- new net N$20: Q6.B, R27.1, R31.1
- new net N$9: R35.2, U9.STAT1
- net 5V: now also D4.C, Q2.S1, R32.1; no longer C33.1, LED10.VDD, LED11.VDD, LED4.VDD, LED7.VDD, LED8.VDD, LED9.VDD, R45.1, R47.1, U5.SENSE
- net CHANNEL_A: now also U1.[PCINT27/TXD1/INT1]_PD3; no longer U1.[PCINT26/RXD1/INT0]_PD2
- net CHANNEL_B: now also U1.[PCINT26/RXD1/INT0]_PD2; no longer U1.[PCINT27/TXD1/INT1]_PD3
- net DISPLAY_POWER: now also Q1.G1, R33.2, TP4.P$1; no longer J2.2, TP40.P$1
- net GND: now also C2.2, C20.2, C22.2, C23.2, C24.2, C30.2, C9.2, D4.A, J5.1, Q6.E, R18.2, R31.2, R5.2, U9.GND; no longer C24.1, C27.1, C28.2, C29.2, C30.1, C31.2, C32.2, C33.2, C5.2, Q1.E, Q6.S, R27.1, R37.1, U12.PGND, U12.SGND
- net N$27: now also U9.PROG; no longer U12.ICHG
- net PWR_IN: now also C23.1, C24.1, Q7.D1; no longer C32.1, C5.1, Q7.S1
- net VBAT: now also C30.1, U9.VBAT1, U9.VBAT2; no longer C27.2, C28.1, C29.1, Q6.G, U12.BAT
- net VBUS_FUSED: now also LED14.+, U9.VDD1, U9.VDD2; no longer C24.2, L1.1, R35.1, R38.2, U12.EN, U12.ILIM
- net VCC: now also Q1.S1, R33.1
- net VIN: now also Q7.S1; no longer Q7.D1
Other:
- note added: "3.7V LI-ION BATTERY CHARGER"
- note added: "DISPLAY POWER CONTROL"
- note added: "LED POWER CONTROL"
- note added: "PROG Resistor: 10K ohm = 100 mA 5K ohm = 200 mA 2.5K ohm = 500 mA 1K ohm = 1000 mA"
- note added: "Set output voltage to 5.2V by swapping R2 (on U5) to 147k ohm"
- note added: "v2.1"
- note removed: "7.4V LI-ION 2S BATTERY CHARGER"
- note removed: "ACCESSORY POWER CONTROL"
- note removed: "Reverse polarity protection"
- note removed: "Trim voltage up to 5.2V"
- note removed: "v2.0"
- moved on the sheet: C1, C10, C2, C21, C23, C24, C25, C26, C30, C6, C7, C8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
